Commit message: add crop and weed

File: parc_robot/urdf/enclosure.xacro (robot description, xacro)
@@ -14,7 +14,7 @@
           <mesh filename="package://parc_robot/meshes/enclosure.stl" scale="0.001 0.001 0.001" />
         </geometry>
-        <!-- <material name="">
+        <material name="">
           <color rgba="0.64706 0.61961 0.58824 1" />
-        </material> -->
+        </material>
       </visual>
       <collision>

File: parc_robot/urdf/sensors.xacro (robot description, xacro)
@@ -4,4 +4,6 @@
   <xacro:include filename="$(find parc_robot)/urdf/ydlidar.xacro" />
   <xacro:include filename="$(find parc_robot)/urdf/zed2.xacro" />
+  <xacro:include filename="$(find parc_robot)/urdf/gps.xacro" />
+  <xacro:include filename="$(find parc_robot)/urdf/side_cameras.xacro" />
   <!-- ydlidar -->
   <xacro:ydlidar_sensor parent="base_link">
@@ -13,3 +15,15 @@
     <origin xyz="0.36 0 0.11" rpy="0 0 0"/>
   </xacro:zed2>
+  <!-- gps -->
+  <xacro:gps_sensor parent="base_link">
+    <origin xyz="0 0 0.2" rpy="0 0 0"/>
+  </xacro:gps_sensor>
+  <!-- left_side_camera -->
+  <xacro:left_side_camera parent="base_link">
+    <origin xyz="0 0.5 0.7" rpy="0 1.0472 1.571428571"/>
+  </xacro:left_side_camera>
+    <!-- right_side_camera -->
+  <xacro:right_side_camera parent="base_link">
+    <origin xyz="0 -0.5 0.7" rpy="0 2.0944 1.571428571"/>
+  </xacro:right_side_camera>
 </robot>

File: parc_robot/urdf/zed2.xacro (robot description, xacro)
@@ -88,4 +88,48 @@
       <xacro:property name="link_prefix" value="${robot_ns}/"/>
     </xacro:if> -->
+    <gazebo reference="zed2_camera_center">
+      <sensor type="camera" name="zed2_center_camera">
+        <always_on>true</always_on>
+        <update_rate>30.0</update_rate>
+        <visualize>false</visualize>
+        <camera name="zed2_center_camera">
+          <horizontal_fov>1.9</horizontal_fov>
+          <image>
+            <width>640</width>
+            <height>480</height>
+            <format>R8G8B8</format>
+          </image>
+          <clip>
+            <near>0.02</near>
+            <far>300</far>
+          </clip>
+          <noise>
+            <type>gaussian</type>
+            <mean>0.0</mean>
+            <stddev>0.007</stddev>
+          </noise>
+          <distortion>
+            <k1>-0.279817</k1>
+            <k2>0.060321</k2>
+            <k3>0.000487</k3>
+            <p1>0.000310</p1>
+            <p2>0.000000</p2>
+            <center>0.5 0.5</center>
+          </distortion>
+        </camera>
+        <plugin name="camera_controller" filename="libgazebo_ros_camera.so">
+          <!-- <robotNamespace>${robot_ns}</robotNamespace> -->
+          <cameraName>camera</cameraName>
+          <imageTopicName>image_raw</imageTopicName>
+          <cameraInfoTopicName>camera_info</cameraInfoTopicName>
+          <frameName>camera_optical_frame</frameName>
+          <distortionK1>-0.279817</distortionK1>
+          <distortionK2>0.060321</distortionK2>
+          <distortionK3>0.000487</distortionK3>
+          <distortionT1>0.000310</distortionT1>
+          <distortionT2>0.000000</distortionT2>
+        </plugin>
+      </sensor>
+    </gazebo>
     <!-- Left/Depth camera -->
     <gazebo reference="zed2_left_camera_frame">
