Commit message: update README.md

File: parc_robot/urdf/attachment.xacro (robot description, xacro)
@@ -5,5 +5,5 @@
   <!-- enclosure -->
   <xacro:enclosure parent="base_link">
-    <origin xyz="0.7 0 0" rpy="0 0 0" />
+    <origin xyz="0.7 0 -0.21" rpy="0 0 0" />
   </xacro:enclosure>
 </robot>

File: parc_robot/urdf/enclosure.xacro (robot description, xacro)
@@ -14,7 +14,7 @@
           <mesh filename="package://parc_robot/meshes/enclosure.stl" scale="0.001 0.001 0.001" />
         </geometry>
-        <material name="">
+        <!-- <material name="">
           <color rgba="0.64706 0.61961 0.58824 1" />
-        </material>
+        </material> -->
       </visual>
       <collision>

Commit message: update seeder and camera attachment

File: parc_robot/urdf/attachment.xacro (robot description, xacro)
@@ -3,7 +3,13 @@
   <!-- Includes -->
   <xacro:include filename="$(find parc_robot)/urdf/enclosure.xacro" />
+  <!-- <xacro:include filename="$(find parc_robot)/urdf/seeder.xacro" /> -->
   <!-- enclosure -->
   <xacro:enclosure parent="base_link">
     <origin xyz="0.7 0 -0.21" rpy="0 0 0" />
   </xacro:enclosure>
+  <!-- seeder -->
+  <!-- <xacro:seeder parent="base_link">
+    <origin xyz="-0.75 0 -0.21" rpy="0 0 0" /> -->
+    <!-- <origin xyz="-0.75 0 -0.21" rpy="0 0 0" /> -->
+  <!-- </xacro:seeder> -->
 </robot>

File: parc_robot/urdf/enclosure.xacro (robot description, xacro)
@@ -9,17 +9,28 @@
         <inertia ixx="6.7885E-05" ixy="-1.3987E-07" ixz="-8.1554E-07" iyy="0.00013173" iyz="-9.0932E-08" izz="7.1972E-05" />
       </inertial>
-      <visual>
+      <visual name="visual">
         <origin xyz="0 0 0" rpy="0 0 0" />
         <geometry>
-          <mesh filename="package://parc_robot/meshes/enclosure.stl" scale="0.001 0.001 0.001" />
+          <!-- <mesh filename="package://parc_robot/meshes/enclosure.dae" scale="0.001 0.001 0.001" /> -->
+          <mesh filename="package://parc_robot/meshes/enclosure_with_overhang.stl" scale="0.001 0.001 0.001" />
         </geometry>
-        <material name="">
+        <!-- <material name="">
           <color rgba="0.64706 0.61961 0.58824 1" />
-        </material>
+        </material> -->
+        <!-- <material name="">
+          <script> -->
+            <!-- <uri>file://parc_robot/materials/scripts/</uri> -->
+            <!-- <uri>file://parc_robot/materials/textures/</uri> -->
+            <!-- <name>dirty_metal</name> -->
+            <!-- <uri>file://media/materials/scripts/gazebo.material</uri>
+            <name>Gazebo/Wood</name>
+          </script>
+        </material> -->
       </visual>
-      <collision>
+      <collision name="collision">
         <origin xyz="0 0 0" rpy="0 0 0" />
         <geometry>
-          <mesh filename="package://parc_robot/meshes/enclosure.stl" scale="0.001 0.001 0.001" />
+          <!-- <mesh filename="package://parc_robot/meshes/enclosure.dae" scale="0.001 0.001 0.001" /> -->
+          <mesh filename="package://parc_robot/meshes/enclosure_with_overhang.stl" scale="0.001 0.001 0.001" />
         </geometry>
       </collision>

File: parc_robot/urdf/sensors.xacro (robot description, xacro)
@@ -21,9 +21,11 @@
   <!-- left_side_camera -->
   <xacro:left_side_camera parent="base_link">
-    <origin xyz="0 0.5 0.7" rpy="0 1.0472 1.571428571"/>
+    <origin xyz="0 0.55 0.635" rpy="0 1.5708 1.571428571"/>
+    <!-- <origin xyz="0 0.7 0.7" rpy="0 1.0472 1.571428571"/> -->
   </xacro:left_side_camera>
     <!-- right_side_camera -->
   <xacro:right_side_camera parent="base_link">
-    <origin xyz="0 -0.5 0.7" rpy="0 2.0944 1.571428571"/>
+    <origin xyz="0 -0.55 0.635" rpy="0 1.5708 1.571428571"/>
+    <!-- <origin xyz="0 -0.7 0.7" rpy="0 2.0944 1.571428571"/> -->
   </xacro:right_side_camera>
 </robot>

Commit message: goal and peg gps coordinates

File: parc_robot/urdf/attachment.xacro (robot description, xacro)
@@ -3,13 +3,7 @@
   <!-- Includes -->
   <xacro:include filename="$(find parc_robot)/urdf/enclosure.xacro" />
-  <!-- <xacro:include filename="$(find parc_robot)/urdf/seeder.xacro" /> -->
   <!-- enclosure -->
   <xacro:enclosure parent="base_link">
     <origin xyz="0.7 0 -0.21" rpy="0 0 0" />
   </xacro:enclosure>
-  <!-- seeder -->
-  <!-- <xacro:seeder parent="base_link">
-    <origin xyz="-0.75 0 -0.21" rpy="0 0 0" /> -->
-    <!-- <origin xyz="-0.75 0 -0.21" rpy="0 0 0" /> -->
-  <!-- </xacro:seeder> -->
 </robot>

File: parc_robot/urdf/enclosure.xacro (robot description, xacro)
@@ -13,17 +13,16 @@
         <geometry>
           <!-- <mesh filename="package://parc_robot/meshes/enclosure.dae" scale="0.001 0.001 0.001" /> -->
-          <mesh filename="package://parc_robot/meshes/enclosure_with_overhang.stl" scale="0.001 0.001 0.001" />
+          <!-- <mesh filename="package://parc_robot/meshes/enclosure_with_overhang.stl" scale="0.001 0.001 0.001" /> -->
+          <mesh filename="package://parc_robot/meshes/enclosure_with_overhang.dae" scale="0.001 0.001 0.001" />
         </geometry>
+        <!-- <material name="dirty_metal">
+          <script>
+            <uri>model://lettuce_crop_01/materials/scripts/</uri>
+            <uri>model://lettuce_crop_01/materials/textures/</uri>
+            <name>dirty_metal</name>
+          </script>
+        </material> -->
         <!-- <material name="">
           <color rgba="0.64706 0.61961 0.58824 1" />
-        </material> -->
-        <!-- <material name="">
-          <script> -->
-            <!-- <uri>file://parc_robot/materials/scripts/</uri> -->
-            <!-- <uri>file://parc_robot/materials/textures/</uri> -->
-            <!-- <name>dirty_metal</name> -->
-            <!-- <uri>file://media/materials/scripts/gazebo.material</uri>
-            <name>Gazebo/Wood</name>
-          </script>
         </material> -->
       </visual>
@@ -32,5 +31,6 @@
         <geometry>
           <!-- <mesh filename="package://parc_robot/meshes/enclosure.dae" scale="0.001 0.001 0.001" /> -->
-          <mesh filename="package://parc_robot/meshes/enclosure_with_overhang.stl" scale="0.001 0.001 0.001" />
+          <!-- <mesh filename="package://parc_robot/meshes/enclosure_with_overhang.stl" scale="0.001 0.001 0.001" /> -->
+          <mesh filename="package://parc_robot/meshes/enclosure_with_overhang.dae" scale="0.001 0.001 0.001" />
         </geometry>
       </collision>
