Commit message: update package

File: parc_robot/urdf/robot.xacro (robot description, xacro)
@@ -56,5 +56,5 @@
     </joint>
     <!-- Scout wheel macros -->
-    <!-- wheel labeled from 0 to 3, conter-clockwise, starting from front right wheel -->
+    <!-- wheel labeled from 0 to 3, counter-clockwise, starting from front right wheel -->
     <!-- motor 1 and 2 (left side) are mechanically installed in a reversed direction -->
     <xacro:scout_wheel_type1 wheel_prefix="front_right">
@@ -72,4 +72,5 @@
     <!-- Sensor definitions -->
     <xacro:include filename="$(find parc_robot)/urdf/sensors.xacro" />
+    <xacro:include filename="$(find parc_robot)/urdf/attachment.xacro" />
     <!-- Gazebo definitions -->
     <xacro:include filename="$(find parc_robot)/urdf/robot_gazebo.xacro" />

File: parc_robot/urdf/robot_gazebo.xacro (robot description, xacro)
@@ -8,59 +8,66 @@
 -->
 <robot xmlns:xacro="http://ros.org/wiki/xacro">
-    <xacro:include filename="$(find parc_robot)/urdf/scout_wheel.gazebo" />
-    <!-- Additional definitions for simulation -->
-    <!-- <gazebo reference="base_link">
-        <material>Gazebo/Grey</material>
-    </gazebo> -->
-    <!-- Actuator configurations -->
-    <xacro:scout_wheel_transmission wheel_prefix="front_right" />
-    <xacro:scout_wheel_transmission wheel_prefix="front_left" />
-    <xacro:scout_wheel_transmission wheel_prefix="rear_left" />
-    <xacro:scout_wheel_transmission wheel_prefix="rear_right" />
-    <!-- Controller configurations -->
-    <!-- <gazebo>
-        <plugin name="gazebo_ros_control" filename="libgazebo_ros_control.so">
-            <robotNamespace>$(arg robot_namespace)</robotNamespace>
-        </plugin>
-    </gazebo> -->
-    <!-- kp spring constant, kd damping constant -->
-    <gazebo>
-        <mu1 value="1.0"/>
-        <mu2 value="0.9"/>
-        <kp value="10000000.0" />
-        <kd value="1.0" />
-        <fdir1 value="1 0 0"/>
-        <minDepth value="0.001" />
-        <maxContacts value="64"/>
-    </gazebo>
-    <gazebo>
-        <plugin name="skid_steer_drive_controller" filename="libgazebo_ros_skid_steer_drive.so">
-            <updateRate>100.0</updateRate>
-            <robotNamespace></robotNamespace>
-            <leftFrontJoint>front_left_wheel</leftFrontJoint>
-            <rightFrontJoint>front_right_wheel</rightFrontJoint>
-            <leftRearJoint>rear_left_wheel</leftRearJoint>
-            <rightRearJoint>rear_right_wheel</rightRearJoint>
-            <wheelSeparation>4</wheelSeparation>
-            <wheelDiameter>0.32918</wheelDiameter>
-            <robotBaseFrame>base_link</robotBaseFrame>
-            <torque>1000</torque>
-            <commandTopic>cmd_vel</commandTopic>
-            <broadcastTF>true</broadcastTF>
-            <odometryTopic>odom</odometryTopic>
-            <odometryFrame>odom</odometryFrame>
-            <covariance_x>0.000100</covariance_x>
-            <covariance_y>0.000100</covariance_y>
-            <covariance_yaw>0.010000</covariance_yaw>
-        </plugin>
-    </gazebo>
-    <!-- <gazebo>
-        <plugin name="object_controller" filename="libgazebo_ros_planar_move.so">
-            <commandTopic>cmd_vel</commandTopic>
-            <odometryTopic>odom</odometryTopic>
-            <odometryFrame>odom</odometryFrame>
-            <odometryRate>20.0</odometryRate>
-            <robotBaseFrame>base_footprint</robotBaseFrame>
-        </plugin>
-    </gazebo> -->
+  <xacro:include filename="$(find parc_robot)/urdf/scout_wheel.gazebo" />
+  <!-- Additional definitions for simulation -->
+  <!-- <gazebo reference="base_link">
+      <material>Gazebo/Grey</material>
+  </gazebo> -->
+  <!-- Actuator configurations -->
+  <xacro:scout_wheel_transmission wheel_prefix="front_right" />
+  <xacro:scout_wheel_transmission wheel_prefix="front_left" />
+  <xacro:scout_wheel_transmission wheel_prefix="rear_left" />
+  <xacro:scout_wheel_transmission wheel_prefix="rear_right" />
+  <!-- Controller configurations -->
+  <gazebo>
+    <plugin name="gazebo_ros_control" filename="libgazebo_ros_control.so">
+			<robotNamespace>/</robotNamespace>
+			<!-- <robotSimType>steer_bot_hardware_gazebo/SteerBotHardwareGazebo</robotSimType> -->
+      <robotSimType>gazebo_ros_control/DefaultRobotHWSim</robotSimType>
+    </plugin>
+  </gazebo>
+	<gazebo>
+    <plugin name="joint_state_publisher" filename="libgazebo_ros_joint_state_publisher.so">
+      <jointName>front_left_wheel, front_right_wheel, rear_left_wheel, rear_right_wheel</jointName>
+    </plugin>
+  </gazebo>
+  <!-- kp spring constant, kd damping constant -->
+  <gazebo>
+    <mu1 value="1.0"/>
+    <mu2 value="0.9"/>
+    <kp value="10000000.0" />
+    <kd value="1.0" />
+    <fdir1 value="1 0 0"/>
+    <minDepth value="0.001" />
+    <maxContacts value="64"/>
+  </gazebo>
+  <gazebo>
+    <plugin name="skid_steer_drive_controller" filename="libgazebo_ros_skid_steer_drive.so">
+      <updateRate>100.0</updateRate>
+      <robotNamespace>/</robotNamespace>
+      <leftFrontJoint>front_left_wheel</leftFrontJoint>
+      <rightFrontJoint>front_right_wheel</rightFrontJoint>
+      <leftRearJoint>rear_left_wheel</leftRearJoint>
+      <rightRearJoint>rear_right_wheel</rightRearJoint>
+      <wheelSeparation>4</wheelSeparation>
+      <wheelDiameter>0.32918</wheelDiameter>
+      <robotBaseFrame>base_link</robotBaseFrame>
+      <torque>1000</torque>
+      <commandTopic>cmd_vel</commandTopic>
+      <broadcastTF>true</broadcastTF>
+      <odometryTopic>odom</odometryTopic>
+      <odometryFrame>odom</odometryFrame>
+      <covariance_x>0.000100</covariance_x>
+      <covariance_y>0.000100</covariance_y>
+      <covariance_yaw>0.010000</covariance_yaw>
+    </plugin>
+  </gazebo>
+  <!-- <gazebo>
+    <plugin name="object_controller" filename="libgazebo_ros_planar_move.so">
+      <commandTopic>cmd_vel</commandTopic>
+      <odometryTopic>odom</odometryTopic>
+      <odometryFrame>odom</odometryFrame>
+      <odometryRate>20.0</odometryRate>
+      <robotBaseFrame>base_footprint</robotBaseFrame>
+    </plugin>
+  </gazebo> -->
 </robot>

File: parc_robot/urdf/sensors.xacro (robot description, xacro)
@@ -6,10 +6,10 @@
   <!-- ydlidar -->
   <xacro:ydlidar_sensor parent="base_link">
-    <origin xyz="0.25 0 0.11" rpy="0 0 0" />
+    <origin xyz="0.25 0 0.13" rpy="0 0 0" />
     <!-- <origin xyz="0.25 0 0.14" rpy="0 0 0" /> -->
   </xacro:ydlidar_sensor>
   <!-- zed2 camera -->
   <xacro:zed2 parent="base_link">
-    <origin xyz="0.35 0 0.11" rpy="0 0 0"/>
+    <origin xyz="0.36 0 0.11" rpy="0 0 0"/>
   </xacro:zed2>
 </robot>

File: parc_robot/urdf/ydlidar.xacro (robot description, xacro)
@@ -44,8 +44,8 @@
     </joint>
     <gazebo reference="${name}_link">
-      <sensor type="gpu_ray" name="${name}_sensor">
+      <sensor type="ray" name="${name}_sensor">
         <pose>0 0 0 0 0 0</pose>
         <visualize>false</visualize>
-        <update_rate>10</update_rate>
+        <update_rate>40</update_rate>
         <ray>
           <scan>
@@ -58,6 +58,6 @@
           </scan>
           <range>
-            <min>0.15</min>
-            <max>6.0</max>
+            <min>0.12</min>
+            <max>16.0</max>
             <resolution>0.01</resolution>
           </range>
@@ -68,5 +68,5 @@
           </noise>
         </ray>
-        <plugin name="gazebo_ros_${name}_controller" filename="libgazebo_ros_gpu_laser.so">
+        <plugin name="gazebo_ros_${name}_controller" filename="libgazebo_ros_laser.so">
           <topicName>/scan</topicName>
           <frameName>${name}_link</frameName>

File: parc_robot/urdf/zed2.xacro (robot description, xacro)
@@ -2,7 +2,7 @@
 <robot xmlns:xacro="http://ros.org/wiki/xacro">
   <xacro:property name="baseline" value="0.12"/>
-  <xacro:macro name="zed2" params="parent *origin link_prefix:='' joint_prefix:=''">
+  <xacro:macro name="zed2" params="parent *origin">
     <!-- Camera Center -->
-    <link name="${link_prefix}zed2_camera_center">
+    <link name="zed2_camera_center">
       <inertial>
         <mass value="0.16140"/>
@@ -25,68 +25,69 @@
     </link>
     <!-- Center Camera -->
-    <joint name="${joint_prefix}zed2_camera_center_joint" type="fixed">
+    <joint name="zed2_camera_center_joint" type="fixed">
       <xacro:insert_block name="origin" />
       <parent link="${parent}"/>
-      <child link="${link_prefix}zed2_camera_center"/>
+      <child link="zed2_camera_center"/>
     </joint>
     <!-- Left Camera -->
-    <joint name="${joint_prefix}zed2_left_camera_joint" type="fixed">
-      <parent link="${link_prefix}zed2_camera_center"/>
-      <child link="${link_prefix}zed2_left_camera_frame"/>
+    <joint name="zed2_left_camera_joint" type="fixed">
+      <parent link="zed2_camera_center"/>
+      <child link="zed2_left_camera_frame"/>
       <origin xyz="0 ${baseline/2} 0" rpy="0 0 0" />
     </joint>
-    <link name="${link_prefix}zed2_left_camera_frame" />
-    <joint name="${joint_prefix}zed2_left_camera_optical_joint" type="fixed">
+    <link name="zed2_left_camera_frame" />
+    <joint name="zed2_left_camera_optical_joint" type="fixed">
       <origin xyz="0 0 0" rpy="-${pi/2} 0.0 -${pi/2}"/>
-      <parent link="${link_prefix}zed2_left_camera_frame"/>
-      <child link="${link_prefix}zed2_left_camera_optical_frame"/>
-    </joint>
-    <link name="${link_prefix}zed2_left_camera_optical_frame"/>
+      <parent link="zed2_left_camera_frame"/>
+      <child link="zed2_left_camera_optical_frame"/>
+    </joint>
+    <link name="zed2_left_camera_optical_frame"/>
     <!-- Right Camera -->
-    <joint name="${joint_prefix}zed2_right_camera_joint" type="fixed">
-      <parent link="${link_prefix}zed2_camera_center"/>
-      <child link="${link_prefix}zed2_right_camera_frame"/>
+    <joint name="zed2_right_camera_joint" type="fixed">
+      <parent link="zed2_camera_center"/>
+      <child link="zed2_right_camera_frame"/>
       <origin xyz="0 -${baseline/2} 0" rpy="0 0 0" />
     </joint>
-    <link name="${link_prefix}zed2_right_camera_frame" />
-    <joint name="${joint_prefix}zed2_right_camera_optical_joint" type="fixed">
+    <link name="zed2_right_camera_frame" />
+    <joint name="zed2_right_camera_optical_joint" type="fixed">
       <origin xyz="0 0 0" rpy="-${pi/2} 0.0 -${pi/2}"/>
-      <parent link="${link_prefix}zed2_right_camera_frame"/>
-      <child link="${link_prefix}zed2_right_camera_optical_frame"/>
-    </joint>
-    <link name="${link_prefix}zed2_right_camera_optical_frame"/>
+      <parent link="zed2_right_camera_frame"/>
+      <child link="zed2_right_camera_optical_frame"/>
+    </joint>
+    <link name="zed2_right_camera_optical_frame"/>
     <!-- Sensors -->
-    <joint name="${joint_prefix}zed2_mag_joint" type="fixed">
-      <parent link="${link_prefix}zed2_camera_center"/>
-      <child link="${link_prefix}zed2_mag_link"/>
+    <joint name="zed2_mag_joint" type="fixed">
+      <parent link="zed2_camera_center"/>
+      <child link="zed2_mag_link"/>
       <origin xyz="0 0 0" rpy="0 0 0" />
     </joint>
-    <link name="${link_prefix}zed2_mag_link" />
-    <joint name="${joint_prefix}zed2_baro_joint" type="fixed">
-      <parent link="${link_prefix}zed2_camera_center"/>
-      <child link="${link_prefix}zed2_baro_link"/>
+    <link name="zed2_mag_link" />
+    <joint name="zed2_baro_joint" type="fixed">
+      <parent link="zed2_camera_center"/>
+      <child link="zed2_baro_link"/>
       <origin xyz="0 0 0" rpy="0 0 0" />
     </joint>
-    <link name="${link_prefix}zed2_baro_link" />
-    <joint name="${joint_prefix}zed2_temp_left_joint" type="fixed">
-      <parent link="${link_prefix}zed2_left_camera_frame"/>
-      <child link="${link_prefix}zed2_temp_left_link"/>
+    <link name="zed2_baro_link" />
+    <joint name="zed2_temp_left_joint" type="fixed">
+      <parent link="zed2_left_camera_frame"/>
+      <child link="zed2_temp_left_link"/>
       <origin xyz="0 0 0" rpy="0 0 0" />
     </joint>
-    <link name="${link_prefix}zed2_temp_left_link" />
-    <joint name="${joint_prefix}zed2_temp_right_joint" type="fixed">
-        <parent link="${link_prefix}zed2_right_camera_frame"/>
-        <child link="${link_prefix}zed2_temp_right_link"/>
+    <link name="zed2_temp_left_link" />
+    <joint name="zed2_temp_right_joint" type="fixed">
+        <parent link="zed2_right_camera_frame"/>
+        <child link="zed2_temp_right_link"/>
         <origin xyz="0 0 0" rpy="0 0 0" />
     </joint>
-    <link name="${link_prefix}zed2_temp_right_link" />
-  </xacro:macro>
-  <xacro:macro name="zed2_gazebo" params="robot_ns:=''">
-    <xacro:property name="link_prefix" value=""/>
+    <link name="zed2_temp_right_link" />
+  <!-- </xacro:macro> -->
+  <!-- <xacro:macro name="zed2_gazebo"> -->
+  <!-- <xacro:macro name="zed2_gazebo" params="robot_ns:=''"> -->
+    <!-- <xacro:property name="link_prefix" value=""/>
     <xacro:if value="${robot_ns != '' and robot_ns != '/'}">
       <xacro:property name="link_prefix" value="${robot_ns}/"/>
-    </xacro:if>
+    </xacro:if> -->
     <!-- Left/Depth camera -->
-    <gazebo reference="${link_prefix}zed2_left_camera_frame">
+    <gazebo reference="zed2_left_camera_frame">
       <!-- Raw images (with lens distortion) -->
       <sensor type="camera" name="zed2_left_raw_camera">
@@ -121,5 +122,5 @@
         </camera>
         <plugin name="camera_controller" filename="libgazebo_ros_camera.so">
-          <robotNamespace>${robot_ns}</robotNamespace>
+          <!-- <robotNamespace>${robot_ns}</robotNamespace> -->
           <cameraName>zed2/left_raw</cameraName>
           <imageTopicName>image_raw_color</imageTopicName>
@@ -160,5 +161,5 @@
         </camera>
         <plugin name="camera_controller" filename="libgazebo_ros_openni_kinect.so">
-          <robotNamespace>${robot_ns}</robotNamespace>
+          <!-- <robotNamespace>${robot_ns}</robotNamespace> -->
           <cameraName>zed2</cameraName>
           <imageTopicName>left/image_rect_color</imageTopicName>
@@ -179,5 +180,5 @@
     </gazebo>
     <!-- Right camera -->
-    <gazebo reference="${link_prefix}zed2_right_camera_frame">
+    <gazebo reference="zed2_right_camera_frame">
       <!-- Raw images (with lens distortion) -->
       <sensor type="camera" name="zed2_right_raw_camera">
@@ -211,5 +212,5 @@
         </camera>
         <plugin name="camera_controller" filename="libgazebo_ros_camera.so">
-          <robotNamespace>${robot_ns}</robotNamespace>
+          <!-- <robotNamespace>${robot_ns}</robotNamespace> -->
           <cameraName>zed2/right_raw</cameraName>
           <imageTopicName>image_raw_color</imageTopicName>
@@ -250,5 +251,5 @@
         </camera>
         <plugin name="camera_controller" filename="libgazebo_ros_camera.so">
-          <robotNamespace>${robot_ns}</robotNamespace>
+          <!-- <robotNamespace>${robot_ns}</robotNamespace> -->
           <cameraName>zed2/right</cameraName>
           <imageTopicName>image_rect_color</imageTopicName>
@@ -263,9 +264,9 @@
     </gazebo>
     <!-- IMU -->
-    <gazebo reference="${link_prefix}zed2_left_camera_frame">
+    <gazebo reference="zed2_left_camera_frame">
       <sensor type="imu" name="zed2_imu_sensor">
         <update_rate>100</update_rate>
         <plugin filename="libgazebo_ros_imu_sensor.so" name="imu_plugin">
-          <robotNamespace>${robot_ns}</robotNamespace>
+          <!-- <robotNamespace>${robot_ns}</robotNamespace> -->
           <topicName>zed2/imu/data</topicName>
           <frameName>zed2_imu_link</frameName>

Commit message: added scout package

File: parc_robot/urdf/robot.xacro (robot description, xacro)
@@ -1,77 +1,9 @@
 <?xml version="1.0"?>
-<robot name="scout_v2"
-    xmlns:xacro="http://ros.org/wiki/xacro">
-    <xacro:arg name="robot_namespace" default="/" />
-    <xacro:include filename="$(find parc_robot)/urdf/scout_wheel_type1.xacro" />
-    <xacro:include filename="$(find parc_robot)/urdf/scout_wheel_type2.xacro" />
-    <!-- Variables -->
-    <xacro:property name="M_PI" value="3.14159"/>
-    <!-- Vehicle Geometries -->
-    <xacro:property name="base_x_size" value="0.9250000" />
-    <xacro:property name="base_y_size" value="0.380000" />
-    <xacro:property name="base_z_size" value="0.210000" />
-    <xacro:property name="wheelbase" value="0.498" />
-    <xacro:property name="track" value="0.58306" />
-    <xacro:property name="wheel_vertical_offset" value="-0.0702" />
-    <xacro:property name="wheel_length" value="1.1653e-01" />
-    <xacro:property name="wheel_radius" value="1.6459e-01" />
-    <!-- Base link -->
-    <link name="base_link">
-        <visual>
-            <origin xyz="0 0 0" rpy="0 0 0" />
-            <geometry>
-                <mesh filename="package://parc_robot/meshes/base_link.dae" />
-            </geometry>
-        </visual>
-        <collision>
-            <origin xyz="0 0 0.008" rpy="0 0 0" />
-            <geometry>
-                <box size="${base_x_size} ${base_y_size} ${base_z_size}"/>
-            </geometry>
-        </collision>
-        <collision>
-            <origin xyz="0 0 ${base_z_size/6}" rpy="0 0 0" />
-            <geometry>
-                <box size="${base_x_size/6} ${base_y_size*1.65} ${base_z_size/3}"/>
-            </geometry>
-        </collision>
-    </link>
-    <link name="base_footprint"/>
-    <joint name="base_footprint_joint" type="fixed">
-        <origin xyz="0 0 ${wheel_vertical_offset - wheel_radius}" rpy="0 0 0" />
-        <parent link="base_link" />
-        <child link="base_footprint" />
-    </joint>
-    <link name="inertial_link">
-        <inertial>
-            <mass value="40" />
-            <origin xyz="0.0 0.0 0.0" />
-            <inertia ixx="2.288641" ixy="0" ixz="0" iyy="5.103976" iyz="0" izz="3.431465" />
-        </inertial>
-    </link>
-    <joint name="inertial_joint" type="fixed">
-        <origin xyz="0 0 0" rpy="0 0 0" />
-        <parent link="base_link" />
-        <child link="inertial_link" />
-    </joint>
-    <!-- Scout wheel macros -->
-    <!-- wheel labeled from 0 to 3, counter-clockwise, starting from front right wheel -->
-    <!-- motor 1 and 2 (left side) are mechanically installed in a reversed direction -->
-    <xacro:scout_wheel_type1 wheel_prefix="front_right">
-        <origin xyz="${wheelbase/2} ${-track/2} ${wheel_vertical_offset}" rpy="3.14 0 0" />
-    </xacro:scout_wheel_type1>
-    <xacro:scout_wheel_type2 wheel_prefix="front_left">
-        <origin xyz="${wheelbase/2} ${track/2} ${wheel_vertical_offset}" rpy="0 0 0" />
-    </xacro:scout_wheel_type2>
-    <xacro:scout_wheel_type1 wheel_prefix="rear_left">
-        <origin xyz="${-wheelbase/2} ${track/2} ${wheel_vertical_offset}" rpy="0 0 0" />
-    </xacro:scout_wheel_type1>
-    <xacro:scout_wheel_type2 wheel_prefix="rear_right">
-        <origin xyz="${-wheelbase/2} ${-track/2} ${wheel_vertical_offset}" rpy="3.14 0 0" />
-    </xacro:scout_wheel_type2>
-    <!-- Sensor definitions -->
-    <xacro:include filename="$(find parc_robot)/urdf/sensors.xacro" />
-    <xacro:include filename="$(find parc_robot)/urdf/attachment.xacro" />
-    <!-- Gazebo definitions -->
-    <xacro:include filename="$(find parc_robot)/urdf/robot_gazebo.xacro" />
+<robot name="scout_v2" xmlns:xacro="http://ros.org/wiki/xacro">
+  <xacro:include filename="$(find scout_description)/urdf/scout_v2.xacro" />
+  <!-- Sensor definitions -->
+  <xacro:include filename="$(find parc_robot)/urdf/sensors.xacro" />
+  <xacro:include filename="$(find parc_robot)/urdf/attachment.xacro" />
+  <!-- Gazebo definitions -->
+  <xacro:include filename="$(find parc_robot)/urdf/robot_gazebo.xacro" />
 </robot>
